File: kicad/buran/buran.kicad_pcb (KiCad board)
At the start: 4 copper layers, 210 x 130 mm, 44 parts, among them IC1 XC6210B332MR, IC2 MAX803SQ308D2T1G, IC3 PCA9952TW_Q900,118, IC4 FT201XS-R, IC5 ATSAMD11D14A-SSNT, J1 M20-9761042, J2 47642-0001, J3 M50-3500542

Commit message: kicad files
Parts:
- removed the ? at (208.3, 30.5)
- removed the ? at (40.6, 142.2)
- removed the ? at (208.3, 142.2)
- removed the REF** at (40.6, 30.5)
- added ?: , , F.Cu at (42.2, 141.7)
- added REF**: MountingHole_4mm_Pad, MountingHole:MountingHole_4mm_Pad, F.Cu at (42.2, 33.0)
- added REF**: MountingHole_4mm_Pad, MountingHole:MountingHole_4mm_Pad, F.Cu at (205.7, 141.9)
- added REF**: MountingHole_4mm_Pad, MountingHole:MountingHole_4mm_Pad, F.Cu at (205.7, 33.1)
Routing:
- net GND: vias 72 -> 79
Other:
- board text added: "Buran 2024"
- board text added: "MountingHole_4mm_Pad"

Commit message: update kicad
Parts:
- removed J2: 47642-0001, SamacSys_Parts:476420001
- added J4: 548190519, SamacSys_Parts:548190519, F.Cu at (126.3, 29.1)
- C1, C2: value C0603C180F5GACTU -> 1uF
- C10, C7: value C0603C180F5GACTU -> 4.7uF
- C3, C9: value C0603C180F5GACTU -> 100nF
- C4, C5: value C0603C180F5GACTU -> 47pF
- C6: value C0603C180F5GACTU -> 10nF
- C8: value C0603C180F5GACTU -> 100nF (0.1uF)
- R14: value 10K -> 4K7
- R4, R5, R6, R7: value 35R -> 30R
Routing:
- net /V_UNREG: track 95.2 -> 93.3 mm
- net GND: vias 79 -> 77

Commit message: modify buran hardware
Connections:
- net /CBUS4 renamed /CBUS4/USART_TX
- net /CBUS5 renamed /CBUS5/USART_RX
Other:
- copper layers 4 -> 2
- board text added: "Buran 2024 - Rev 2"
- board text added: "CBUS0"
- board text added: "CBUS1"
- board text added: "CBUS2"
- board text added: "CBUS3"
- board text added: "CBUS4/USART_TX"
- board text added: "CBUS5/USART_RX"
- board text added: "GND"
- board text added: "N_RESET"
- board text added: "SCL"
- board text added: "SDA"
- board text added: "VDD"
- board text added: "V_UNREG"
- board text removed: "Buran 2024"

Commit message: reference files for v3.0
Parts:
- removed the ? at (42.2, 141.7)
- removed C4: 47pF, SamacSys_Parts:CAPC1608X87N
- removed the C5 at (121.4, 32.5)
- removed the C6 at (133.6, 27.9)
- removed C7: 4.7uF, SamacSys_Parts:CAPC1608X87N
- removed C8: 100nF (0.1uF), SamacSys_Parts:CAPC1608X87N
- removed IC3: PCA9952TW_Q900,118, SamacSys_Parts:SOP65P640X110-29N
- removed the IC4 at (125.0, 46.2)
- removed R10: 27R, SamacSys_Parts:ERA3AEB101V
- removed R11: 100K, SamacSys_Parts:ERA3AEB101V
- removed R12, R13: 4K7, SamacSys_Parts:ERA3AEB101V
- removed REF** (x3): MountingHole_4mm_Pad, MountingHole:MountingHole_4mm_Pad
- added ?: , , F.Cu at (166.2, 25.8)
- added ? (x2): , , F.Cu at (38.8, 122.2)
- added ?: , , F.Cu at (166.0, 123.0)
- added ?: , , F.Cu at (39.0, 25.0)
- added J2: M20-7820946, SamacSys_Parts:RHDR9W70P0X254_1X9_2326X250X865P, F.Cu at (100.1, 17.4)
- J3: value M50-3500542 -> M20-7820946; footprint SamacSys_Parts:M503500542 -> SamacSys_Parts:RHDR9W70P0X254_1X9_2326X250X865P
- J4: value 548190519 -> TC2030-CTX-NL; footprint SamacSys_Parts:548190519 -> SamacSys_Parts:TC2030MCPNL10
- MCU LED 1: renamed from LED_MCU_1
- MCU LED 2: renamed from LED_MCU_2
- POWER : renamed from LED_POWER1
- R8: value 2K8 -> 30R
- R9: value 27R -> 30R
- moved POWER  122.4 mm to (43.7, 31.4)
- moved MCU LED 2 122.4 mm to (68.1, 31.4)
- moved R3 122.4 mm to (68.1, 35.0)
- moved MCU LED 1 122.4 mm to (55.9, 31.4)
- moved R2 122.4 mm to (55.9, 35.0)
- moved R1 122.2 mm to (43.9, 35.2)
- moved R9 86.5 mm to (114.0, 122.0), turned to 0 degrees
- moved C3 51.6 mm to (86.7, 43.9)
- moved IC2 51.5 mm to (83.1, 44.2)
- moved C1 51.2 mm to (97.2, 57.2), turned to -90 degrees
- moved J3 50.9 mm to (115.6, 17.4)
- moved R7 50.3 mm to (138.0, 116.0), turned to 0 degrees
- moved S5 46.8 mm to (147.6, 51.8), turned to 180 degrees
- moved IC1 44.9 mm to (101.7, 57.2), turned to 0 degrees
- moved J4 42.2 mm to (145.0, 67.0), turned to 0 degrees
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- renumbered C9 to C5, C10 to C6, IC5 to IC4
Connections:
- C2 pad 2: VDD -> /V_LEDs
- IC1 pad 5: VDD -> /V_LEDs
- IC4 pad 10: /CBUS5/USART_RX -> /USART_RX
- IC4 pad 14: /MCU_S1 -> /MCU_S2
- IC4 pad 15: /MCU_S2 -> /MCU_S1
- IC4 pad 20: /MCU_N_OE -> /MCU_DBG_5
- IC4 pad 3: /CBUS0 -> /MCU_DBG_4
- IC4 pad 4: /CBUS1 -> /MCU_DBG_3
- IC4 pad 5: /CBUS2 -> /MCU_DBG_2
- IC4 pad 8: /CBUS3 -> /MCU_DBG_1
- IC4 pad 9: /CBUS4/USART_TX -> /USART_TX
- J1 pad 11: /CBUS0 -> unconnected-(J1-Pad11)
- J1 pad 12: unconnected-(J1-Pad12) -> /MCU_DBG_5
- J1 pad 13: /CBUS1 -> /N_RESET
- J1 pad 14: unconnected-(J1-Pad14) -> /MCU_DBG_4
- J1 pad 15: /CBUS2 -> unconnected-(J1-Pad15)
- J1 pad 16: unconnected-(J1-Pad16) -> /MCU_DBG_3
- J1 pad 17: /CBUS3 -> /USART_RX
- J1 pad 18: unconnected-(J1-Pad18) -> /MCU_DBG_2
- J1 pad 19: /CBUS4/USART_TX -> /USART_TX
- J1 pad 20: unconnected-(J1-Pad20) -> /MCU_DBG_1
- J1 pad 4: /CBUS5/USART_RX -> unconnected-(J1-Pad4)
- J1 pad 5: /SDA -> unconnected-(J1-Pad5)
- J1 pad 7: /SCL -> unconnected-(J1-Pad7)
- J1 pad 9: /N_RESET -> unconnected-(J1-Pad9)
- J3 pad 1: VDD -> unconnected-(J3-Pad1)
- J3 pad 2: /SWDIO -> unconnected-(J3-Pad2)
- J3 pad 4: /SWCLK -> unconnected-(J3-Pad4)
- J3 pad 5: GND -> /USART_TX
- J3 pad 9: unconnected-(J3-Pad9) -> /USART_RX
- J4 pad 1: /V_UNREG -> VDD
- J4 pad 2: /D0- -> /SWDIO
- J4 pad 3: /D0+ -> /N_RESET
- J4 pad 4: GND -> /SWCLK
- R4 pad 1: /IC4_LED_0 -> GND
- R5 pad 1: /IC4_LED_3 -> GND
- R5 pad 2: Net-(S2-L1) -> Net-(S2-L4)
- R6 pad 1: /IC4_LED_6 -> GND
- R6 pad 2: Net-(S3-L1) -> Net-(S4-L1)
- R7 pad 1: /IC4_LED_9 -> GND
- R7 pad 2: Net-(S4-L1) -> Net-(S4-L4)
- R8 pad 2: Net-(IC3-REXT) -> Net-(S4-L3)
- R9 pad 1: /D0- -> GND
- R9 pad 2: /D- -> Net-(S3-L3)
- S1 pad 4: VDD -> /V_LEDs
- S1 pad 6: /IC4_LED_1 -> /V_LEDs
- S1 pad 7: /IC4_LED_2 -> /V_LEDs
- S2 pad 4: VDD -> /V_LEDs
- S2 pad 5: Net-(S2-L1) -> /V_LEDs
- S2 pad 6: /IC4_LED_4 -> Net-(S2-L4)
- S2 pad 7: /IC4_LED_5 -> /V_LEDs
- S3 pad 4: VDD -> /V_LEDs
- S3 pad 5: Net-(S3-L1) -> /V_LEDs
- S3 pad 6: /IC4_LED_7 -> /V_LEDs
- S3 pad 7: /IC4_LED_8 -> Net-(S3-L3)
- S4 pad 4: VDD -> /V_LEDs
- S4 pad 6: /IC4_LED_10 -> Net-(S4-L4)
- S4 pad 7: /IC4_LED_11 -> Net-(S4-L3)
Routing:
- net VDD: track 522.5 -> 192.9 mm
- net /V_LEDs: track 0.00 -> 293.9 mm
- net /USART_TX: track 0.00 -> 114.4 mm, vias 0 -> 3
- net /USART_RX: track 0.00 -> 104.0 mm, vias 0 -> 3
- net /SCL: track 94.3 -> 0.00 mm, vias 3 -> 0
- net /SDA: track 93.5 -> 0.00 mm, vias 2 -> 0
- net /IC4_LED_11: track 90.3 -> 0.00 mm, vias 2 -> 0
- net /CBUS4/USART_TX: track 89.8 -> 0.00 mm, vias 7 -> 0
- net /IC4_LED_2: track 85.0 -> 0.00 mm
- net /IC4_LED_10: track 83.8 -> 0.00 mm, vias 2 -> 0
- net /IC4_LED_1: track 83.2 -> 0.00 mm
- net /CBUS3: track 81.3 -> 0.00 mm, vias 6 -> 0
- net /CBUS5/USART_RX: track 77.9 -> 0.00 mm, vias 3 -> 0
- net /IC4_LED_9: track 74.4 -> 0.00 mm
- net /CBUS2: track 69.8 -> 0.00 mm, vias 7 -> 0
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Other:
- board size 210 x 130 mm -> 150.7 x 120.7 mm
- board text added: "Buran - 2024"
- board text added: "MCU_DBG_1"
- board text added: "MCU_DBG_2"
- board text added: "MCU_DBG_3"
- board text added: "MCU_DBG_4"
- board text added: "MCU_DBG_5"
- board text added: "USART_RX"
- board text added: "USART_TX"
- board text removed: "CBUS0"
- board text removed: "CBUS1"
- board text removed: "CBUS2"
- board text removed: "CBUS3"
- board text removed: "CBUS4/USART_TX"
- board text removed: "CBUS5/USART_RX"
- board text removed: "SCL"
- board text removed: "SDA"
