File: kicad/buran/buran.kicad_sch (KiCad schematic)
At the start: 40 parts, among them IC1 XC6210B332MR, IC2 MAX803SQ308D2T1G, IC3 PCA9952TW_Q900,118, IC4 FT201XS-R, IC5 ATSAMD11D14A-SSNT, J1 M20-9761042, J2 47642-0001, J3 M50-3500542

Commit message: kicad files
Parts:
- C1, C2: value C0603C180F5GACTU -> 1uF
- C10, C7: value C0603C180F5GACTU -> 4.7uF
- C3, C9: value C0603C180F5GACTU -> 100nF
- C4, C5: value C0603C180F5GACTU -> 47pF
- C6: value C0603C180F5GACTU -> 10nF
- C8: value C0603C180F5GACTU -> 100nF (0.1uF)
- R14: value 10K -> 4K7
- R4, R5, R6, R7: value 35R -> 30R
Other:
- moved on the sheet: C4

Commit message: update kicad
Parts:
- removed J2: 47642-0001, SamacSys_Parts:476420001, symbol SamacSys:47642-0001
- added J4: 548190519, SamacSys_Parts:548190519, symbol SamacSys:548190519
Connections:
- net D0+: now also J4.3 (D+)
- net D0-: now also J4.2 (D-)
- net GND: now also J4.4 (ID), J4.5 (GND), J4.MH1, J4.MH2
- net V_UNREG: now also J4.1 (VBUS)
- no-connect marks 17 -> 16
Other:
- moved on the sheet: R10, R9

Commit message: modify buran hardware
Connections:
- net CBUS4: no longer IC5.9 (PA22)
- net CBUS5: no longer IC5.10 (PA23)
- new net CBUS4/USART_TX: IC5.9 (PA22)
- new net CBUS5/USART_RX: IC5.10 (PA23)
Changed lines of the file:
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@@
-    (stroke (width 0) (type default))
-  )
-  (wire (pts (xy 289.56 86.36) (xy 300.99 86.36))
     (stroke (width 0) (type default))
   )
@@
     (stroke (width 0) (type default))
   )
-  (wire (pts (xy 271.78 76.2) (xy 276.86 76.2))
+  (wire (pts (xy 270.51 76.2) (xy 276.86 76.2))
     (stroke (width 0) (type default))
   )
@@
     (stroke (width 0) (type default))
   )
+  (wire (pts (xy 270.51 86.36) (xy 300.99 86.36))
+    (stroke (width 0) (type default))
+  )
   (wire (pts (xy 233.68 77.47) (xy 243.84 77.47))
     (stroke (width 0) (type default))
@@
     (stroke (width 0) (type default))
   )
-  (wire (pts (xy 271.78 78.74) (xy 285.75 78.74))
+  (wire (pts (xy 270.51 78.74) (xy 285.75 78.74))
     (stroke (width 0) (type default))
   )
@@
     (stroke (width 0) (type default))
   )
-  (wire (pts (xy 289.56 83.82) (xy 300.99 83.82))
+  (wire (pts (xy 270.51 83.82) (xy 300.99 83.82))
     (stroke (width 0) (type default))
   )
@@
   (wire (pts (xy 285.75 236.22) (xy 288.29 236.22))
     (stroke (width 0) (type default))
+  )
+  (text_box "See page 13 ATSAMD11 Reference Manual\nPA22 - SERCOM1[0]\nPA23 - SERCOM1[1]"
+    (at 270.51 87.63 0) (size 25.4 10.16)
+    (stroke (width 0) (type default))
+    (fill (type none))
+    (effects (font (size 1.27 1.27)) (justify left top))
   )
   (text_box "For R8 see Section 7.3.15.1 - Adjusting output peak current\n"
@@
     (effects (font (size 1.27 1.27)) (justify left bottom))
   )
-  (label "SCL" (at 271.78 78.74 0) (fields_autoplaced)
+  (label "SCL" (at 270.51 78.74 0) (fields_autoplaced)
     (effects (font (size 1.27 1.27)) (justify left bottom))
   )
@@
     (effects (font (size 1.27 1.27)) (justify left bottom))
   )
-  (label "CBUS5" (at 289.56 86.36 0) (fields_autoplaced)
+  (label "CBUS5{slash}USART_RX" (at 270.51 86.36 0) (fields_autoplaced)
     (effects (font (size 1.27 1.27)) (justify left bottom))
   )
@@
     (effects (font (size 1.27 1.27)) (justify left bottom))
   )
-  (label "CBUS4" (at 289.56 83.82 0) (fields_autoplaced)
+  (label "CBUS4{slash}USART_TX" (at 270.51 83.82 0) (fields_autoplaced)
     (effects (font (size 1.27 1.27)) (justify left bottom))
   )
@@
     (effects (font (size 1.27 1.27)) (justify left bottom))
   )
-  (label "SDA" (at 271.78 76.2 0) (fields_autoplaced)
-    (effects (font (size 1.27 1.27)) (justify left bottom))
-  )
+  (label "SDA" (at 270.51 76.2 0) (fields_autoplaced)
+    (effects (font (size 1.27 1.27)) (justify left bottom))
+  )

Commit message: reference files for v3.0
Parts:
- removed C4, C5: 47pF, SamacSys_Parts:CAPC1608X87N, symbol SamacSys:C0603C180F5GACTU
- removed C6: 10nF, SamacSys_Parts:CAPC1608X87N, symbol SamacSys:C0603C180F5GACTU
- removed C8: 100nF (0.1uF), SamacSys_Parts:CAPC1608X87N, symbol SamacSys:C0603C180F5GACTU
- removed IC4: FT201XS-R, SamacSys_Parts:SOP64P599X175-16N, symbol SamacSys:FT201XS-R
- removed J3: M50-3500542, SamacSys_Parts:M503500542, symbol SamacSys:M50-3500542
- removed J4: 548190519, SamacSys_Parts:548190519, symbol SamacSys:548190519
- removed R10: 27R, SamacSys_Parts:ERA3AEB101V, symbol SamacSys:ERA3AEB471V
- added J2, J3: M20-7820946, SamacSys_Parts:RHDR9W70P0X254_1X9_2326X250X865P, symbol SamacSys:M20-7820946
- added J4: TC2030-CTX-NL, SamacSys_Parts:TC2030MCPNL10, symbol SamacSys:TC2030-CTX-NL
- added R8: 25R, SamacSys_Parts:ERA3AEB101V, symbol SamacSys:ERA3AEB471V
- C4: renamed from C7; now not fitted
- IC3, R11, R12, R13: now not fitted
- R10: renamed from R8; now not fitted
- R4, R6: value 30R -> 35R
- R5, R7: value 30R -> 25R
- R9: value 27R -> 25R
- renumbered C9 to C5, C10 to C6, IC5 to IC4
Connections:
- net CBUS4/USART_TX is gone; now on net USART_TX: IC4.9 (PA22)
- net CBUS5/USART_RX is gone; now on net USART_RX: IC4.10 (PA23)
- net D0- is gone; now on net GND: R9.1
- net GND: now also R4.1, R5.1, R6.1, R7.1, J2.9, J3.3, J4.5, R8.1
- net IC4_LED_0: no longer R4.1
- net IC4_LED_1: no longer S1.6 (L4)
- net IC4_LED_10: no longer S4.6 (L4)
- net IC4_LED_11: no longer S4.7 (L3)
- net IC4_LED_2: no longer S1.7 (L3)
- net IC4_LED_3: no longer R5.1
- net IC4_LED_4: no longer S2.6 (L4)
- net IC4_LED_5: no longer S2.7 (L3)
- net IC4_LED_6: no longer R6.1
- net IC4_LED_7: no longer S3.6 (L4)
- net IC4_LED_8: no longer S3.7 (L3)
- net IC4_LED_9: no longer R7.1
- net MCU_N_OE: no longer IC4.20 (PA04)
- net MCU_S1: now also IC4.15 (PA25); no longer IC4.14 (PA24)
- net MCU_S2: now also IC4.14 (PA24); no longer IC4.15 (PA25)
- net N_RESET: now also J1.13, J4.3; no longer J1.9
- net SCL: no longer J1.7
- net SDA: no longer J1.5
- net SWCLK: now also J4.4
- net SWDIO: now also J4.2
- net VDD: now also J2.5, J4.1; no longer C2.2, IC1.5 (VOUT), S1.4 (L2), S2.4 (L2), S3.4 (L2), S4.4 (L2)
- net V_UNREG: now also J2.6
- net at R7.2: now also S4.6 (L4); no longer S4.5 (L1)
- net MCU_DBG_5: now reaches J1.12
- net MCU_DBG_5: now also IC4.20 (PA04)
- net MCU_DBG_4: now reaches J1.14
- net MCU_DBG_4: now also IC4.3 (PA07)
- net MCU_DBG_3: now reaches J1.16
- net MCU_DBG_3: now also IC4.4 (PA08)
- net MCU_DBG_2: now reaches J1.18
- net MCU_DBG_2: now also IC4.5 (PA09)
- net MCU_DBG_1: now reaches J1.20
- net MCU_DBG_1: now also IC4.8 (PA16)
- net at R6.2: now also S4.5 (L1); no longer S3.5 (L1)
- net at R5.2: now also S2.6 (L4); no longer S2.5 (L1)
- net CBUS0: no longer names the net of J1.11
- net CBUS0: no longer IC4.3 (PA07)
- removed net CBUS1: IC4.4 (PA08), J1.13
- net CBUS2: no longer names the net of J1.15
- net CBUS2: no longer IC4.5 (PA09)
- net CBUS3 renamed USART_RX
- net USART_RX: now also J3.9; no longer IC4.8 (PA16)
- net CBUS4 renamed USART_TX
- net USART_TX: now also J3.5
- net CBUS5: no longer names the net of J1.4
- net D-: no longer names the net of R9.2
- net D-: now also S3.7 (L3)
- new net: R8.2, S4.7 (L3)
- new net V_LEDs: C2.2, IC1.5 (VOUT), S1.4 (L2), S1.6 (L4), S1.7 (L3), S2.4 (L2), S2.5 (L1), S2.7 (L3), S3.4 (L2), S3.5 (L1), S3.6 (L4), S4.4 (L2)
- no-connect marks 16 -> 26
Other:
- note added: "FTDI MODULE HEADERS"
- note added: "RGB LED DRIVER (NOT INCLUDED)"
- note removed: "FTDI CHIP + USB HEADER"
- note removed: "FTDI Chip"
- note removed: "RGB LED DRIVER"
- note removed: "USB Header"
- moved on the sheet: S3, S4
